File: esp_32_dev_board.sch (KiCad schematic (older format))
At the start: 27 parts, among them J1 Conn_01x19_Male, J2 Conn_01x19_Male, U1 Symbol, U2 ESP32_IC, U3 Flash

Commit message: second commit included some footprins
Parts:
- ANT1: footprint (none) -> RF_Antenna:Texas_SWRA117D_2.4GHz_Right
- C1, C10, C11, C16, C17, C18, C19, C2, C20, C3, C4, C5, C6, C9: footprint (none) -> Capacitor_SMD:C_01005_0402Metric
- C12: footprint (none) -> Resistor_SMD:R_0603_1608Metric
- C13: footprint (none) -> Capacitor_SMD:C_0201_0603Metric
- C14: footprint (none) -> esp32_dev_board:C14_GRM1555C1H4R7BA01D
- C15: footprint (none) -> esp32_dev_board:C15_GRM1555C1H2R4CA01D
- D1: footprint (none) -> esp32_dev_board:DIODFN2_98X58X50L26X51N
- J1, J2: footprint (none) -> TerminalBlock_Altech:Altech_AK300_1x19_P5.00mm_45-Degree
- L4: footprint (none) -> esp32_dev_board:L4_LQP15MN2N4B02D
- R1: footprint (none) -> Resistor_SMD:R_0402_1005Metric
- U1: footprint (none) -> Crystal:Crystal_SMD_3225-4Pin_3.2x2.5mm_HandSoldering
- U2: footprint (none) -> esp32_dev_board:QFN35P500X500X90-49N
- U3: footprint (none) -> esp32_dev_board:GD25Q32
