File: Esp32C_v4_Devkit/Esp32_v4_board.sch (KiCad schematic (older format))
At the start: 34 parts, among them J1 USB_CON8, J2 Conn_01x19_Male, J3 Conn_01x19_Male, Q1 SS8O5O-G, Q2 SS8O5O-G, SW1 SW_Push, SW2 SW_Push, U1 CP2102N-A01-GQFN28, U2 AMS117_3.3

Commit message: Updated board
Parts:
- J1: symbol ESP32-WROOM-32D:USB_CON8 -> Esp32_v4_board-rescue:USB_CON8-ESP32-WROOM-32D
Changed lines of the file:
@@
 	6900 9825 6900 10175
 $Comp
-L ESP32-WROOM-32D:USB_CON8 J1
+L Esp32_v4_board-rescue:USB_CON8-ESP32-WROOM-32D J1
 U 1 1 6072CD8E
 P 2300 5875
